Commit message: Updated collision for custom head

File: tiago_description/urdf/head/head_custom.urdf.xacro (robot description, xacro)
@@ -47,5 +47,5 @@
         <origin xyz="0.0 0 0" rpy="0 0 0.0" />
         <geometry>
-          <mesh filename="package://tiago_description/meshes/head/head_1_custom.stl" scale="1 1 1"/>
+          <mesh filename="package://tiago_description/meshes/head/head_1_custom_collision.dae" scale="1 1 1"/>
         </geometry>
         <material name="White" />
@@ -87,5 +87,5 @@
         <origin xyz="0 0 0" rpy="0 0 0" />
         <geometry>
-          <mesh filename="package://tiago_description/meshes/head/head_2_custom.stl" scale="1 1 1"/>
+          <mesh filename="package://tiago_description/meshes/head/head_2_custom_collision.dae" scale="1 1 1"/>
         </geometry>
       </collision>

File: tiago_description/urdf/sensors/azure_kinect.urdf.xacro (robot description, xacro)
@@ -46,10 +46,10 @@
         </material>
       </visual>
-      <collision>
+      <!-- <collision>
         <origin xyz="0 0 0" rpy="0 0 0"/>
         <geometry>
           <mesh filename="package://tiago_description/meshes/sensors/azure_kinect.stl" />
         </geometry>
-      </collision>
+      </collision> -->
     </link>
     <!-- Gazebo config -->
