Commit message: Azure Kinect URDF complete with correct naming

File: tiago_description/robots/tiago.urdf.xacro (robot description, xacro)
@@ -25,4 +25,6 @@
   <!-- pmb2, omni_base -->
   <xacro:arg name="base_type" default="pmb2"/>
+  <!-- original, custom -->
+  <xacro:arg name="head_type" default="custom"/>
   <!-- no-laser, hokuyo, sick-551, sick-561, sick-571-->
   <xacro:arg name="laser_model" default="sick-571"/>
@@ -38,5 +40,7 @@
   <xacro:arg name="end_effector" default="pal-hey5"/>
   <!-- no-camera, orbbec-astra, orbbec-astra-pro, asus-xtion -->
-  <xacro:arg name="camera_model" default="orbbec-astra"/>
+  <xacro:arg name="camera_model" default="azure-kinect"/>
+  <!-- no-add-on, lidar-back -->
+  <xacro:arg name="add_on_module" default="lidar-back"/>
   <!-- false, true -->
   <xacro:arg name="has_thermal_camera" default="false"/>
@@ -54,4 +58,5 @@
   <!-- HW configuration -->
   <xacro:property name="base_type" value="$(arg base_type)" />
+  <xacro:property name="head_type" value="$(arg head_type)" />
   <xacro:property name="laser_model" value="$(arg laser_model)" />
   <xacro:property name="arm_type" value="$(arg arm_type)" />
@@ -63,7 +68,11 @@
   <xacro:property name="has_screen" value="$(arg has_screen)" />
   <xacro:property name="no_safety_eps" value="$(arg no_safety_eps)" />
+  <xacro:property name="add_on_module" value="$(arg add_on_module)" />
   <!-- HW configuration check -->
   <xacro:if value="${base_type not in ['pmb2', 'omni_base']}">
     <xacro:wrong_base_type/>
+  </xacro:if>
+  <xacro:if value="${head_type not in ['original', 'custom']}">
+    <xacro:wrong_head_type/>
   </xacro:if>
   <xacro:if value="${laser_model not in ['no-laser', 'sick-551', 'sick-561', 'sick-571', 'hokuyo']}">
@@ -82,6 +91,9 @@
     <xacro:wrong_end_effector/>
   </xacro:if>
-  <xacro:if value="${camera_model not in ['no-camera', 'orbbec-astra', 'orbbec-astra-pro', 'asus-xtion']}">
+  <xacro:if value="${camera_model not in ['no-camera', 'orbbec-astra', 'orbbec-astra-pro', 'asus-xtion', 'azure-kinect']}">
     <xacro:wrong_camera_model/>
+  </xacro:if>
+  <xacro:if value="${add_on_module not in ['no-add-on', 'lidar-back']}">
+    <xacro:wrong_add_on_module/>
   </xacro:if>
   <!-- HW configuration helpers-->
@@ -126,5 +138,10 @@
   </xacro:if>
   <!-- Head -->
-  <xacro:include filename="$(find tiago_description)/urdf/head/head.urdf.xacro" />
+  <xacro:if value="${head_type == 'original'}">
+    <xacro:include filename="$(find tiago_description)/urdf/head/head.urdf.xacro" />
+  </xacro:if>
+  <xacro:if value="${head_type == 'custom'}">
+    <xacro:include filename="$(find tiago_description)/urdf/head/head_custom.urdf.xacro" />
+  </xacro:if>
   <!-- Materials for visualization -->
   <xacro:include filename="$(find pal_urdf_utils)/urdf/materials.urdf.xacro" />
@@ -134,5 +151,5 @@
   <!-- Base -->
   <xacro:if value="${base_type == 'pmb2'}">
-    <xacro:base_sensors name="base" laser_model="${laser_model}" has_sonars="true" has_microphone="true"/>
+    <xacro:base_sensors name="base" laser_model="${laser_model}" has_sonars="true" has_microphone="true" add_on_module="${add_on_module}"/>
   </xacro:if>
   <xacro:if value="${base_type == 'omni_base'}">

File: tiago_description/urdf/head/head_custom.urdf.xacro (robot description, xacro)
@@ -25,6 +25,5 @@
   <!-- INCLUDES -->
   <xacro:include filename="$(find pal_urdf_utils)/urdf/deg_to_rad.urdf.xacro" />
-  <xacro:include filename="$(find tiago_description)/urdf/sensors/xtion_pro_live.urdf.xacro" />
-  <xacro:include filename="$(find tiago_description)/urdf/sensors/orbbec_astra.urdf.xacro" />
+  <xacro:include filename="$(find tiago_description)/urdf/sensors/azure_kinect.urdf.xacro" />
   <xacro:include filename="$(arg description_calibration_dir)/calibration_constants.urdf.xacro" />
   <!-- MACRO DEFINITION-->
@@ -50,5 +49,5 @@
         </geometry>
         <material name="White" />
-      </collision>
+      </collision>Head
     </link>
     <joint name="${name}_joint" type="revolute">
@@ -73,13 +72,12 @@
     <link name="${name}_link">
       <inertial>
-        <origin xyz="0.04700 0.05542 0.00022" rpy="0.00000 0.00000 0.00000"/>
-        <mass value="0.66123"/>
-        <!-- Only 0.378 kg of plastic cover, remaining is motor (0.28323) -->
-        <inertia ixx="0.00462000000" ixy="0.00068900000" ixz="0.00000600000" iyy="0.00486100000" iyz="0.00000600000" izz="0.00313200000"/>
+        <origin xyz="0.007999 0.000235 -0.024779" rpy="0.00000 0.00000 0.00000"/>
+        <mass value="0.188"/>
+        <inertia ixx="0.000864253" ixy="-9.286e-11" ixz="6.0e-9" iyy="0.000422887" iyz="-4.13e-7" izz="0.000538406"/>
       </inertial>
       <visual>
         <origin xyz="0 0 0" rpy="0 0 0" />
         <geometry>
-          <mesh filename="package://tiago_description/meshes/head/head_2.stl" scale="1 1 1"/>
+          <mesh filename="package://tiago_description/meshes/head/azure_kinect_mount.stl" scale="1 1 1"/>
         </geometry>
         <material name="White" />
@@ -88,5 +86,5 @@
         <origin xyz="0 0 0" rpy="0 0 0" />
         <geometry>
-          <mesh filename="package://tiago_description/meshes/head/head_2_collision.dae" scale="1 1 1"/>
+          <mesh filename="package://tiago_description/meshes/head/azure_kinect_mount.stl" scale="1 1 1"/>
         </geometry>
       </collision>
@@ -107,36 +105,9 @@
     <xacro:head_1 name="${name}_1" parent="${parent}" />
     <xacro:head_2 name="${name}_2" parent="${name}_1_link"/>
-    <!-- Cameras-->
-    <!-- Asus Xtion-->
-    <xacro:if value="${camera_model == 'asus-xtion'}">
-      <xacro:xtion_pro_live name="head_front_camera" parent="${name}_2_link" camera_model="${camera_model}" extrinsic_calibration_dir="${extrinsic_calibration_dir}">
-        <origin xyz="${camera_position_x} ${camera_position_y} ${camera_position_z}" rpy="${camera_orientation_r} ${camera_orientation_p} ${camera_orientation_y}" />
-        <!-- optical origin -->
-        <origin xyz="0 0 0" rpy="${-90 * deg_to_rad} ${0 * deg_to_rad} ${-90 * deg_to_rad}" />
-      </xacro:xtion_pro_live>
-    </xacro:if>
-    <!-- Orbecc Astra-->
-    <xacro:if value="${camera_model in ['orbbec-astra', 'orbbec-astra-pro']}">
-      <xacro:orbbec_astra name="head_front_camera" parent="${name}_2_link" camera_model="${camera_model}" extrinsic_calibration_dir="${extrinsic_calibration_dir}">
-        <origin xyz="${camera_position_x} ${camera_position_y} ${camera_position_z}" rpy="${camera_orientation_r} ${camera_orientation_p} ${camera_orientation_y}" />
-        <!-- optical origin -->
-        <origin xyz="0 0 0" rpy="${-90 * deg_to_rad} ${0 * deg_to_rad} ${-90 * deg_to_rad}" />
-      </xacro:orbbec_astra>
-    </xacro:if>
-    <!-- Thermal camera -->
-    <xacro:if value="${has_thermal_camera}">
-      <joint name="thermal_camera_joint" type="fixed">
-        <parent link="${head_link_name}"/>
-        <child link="thermal_camera"/>
-        <origin xyz="0.05 0.15 0" rpy="${0*deg_to_rad} ${-90*deg_to_rad} ${-180*deg_to_rad}" />
-      </joint>
-      <link name="thermal_camera">
-        <inertial>
-          <origin xyz="0 0 0" rpy="0 0 0"/>
-          <mass value="0.0001" />
-          <inertia ixx="0.0001" ixy="0" ixz="0" iyy="0.0001" iyz="0" izz="0.0001" />
-        </inertial>
-      </link>
-    </xacro:if>
+    <!-- Azure Kinect -->
+    <!-- CHECK VALUES FROM CAMERA REAL NODE -->
+    <xacro:azure_kinect name="azure_kinect" parent="${name}_2_link" xyz="-0.008 0.097 0" rpy="${-90 * deg_to_rad} 0.0 0.0" >
+    <!-- Parent link frame to Kinect Screw Mount -->
+    </xacro:azure_kinect>
   </xacro:macro>
 </robot>

Commit message: Fix head 1 origin and sim

File: tiago_description/robots/tiago.urdf.xacro (robot description, xacro)
@@ -40,5 +40,5 @@
   <xacro:arg name="end_effector" default="pal-hey5"/>
   <!-- no-camera, orbbec-astra, orbbec-astra-pro, asus-xtion -->
-  <xacro:arg name="camera_model" default="azure-kinect"/>
+  <xacro:arg name="camera_model" default="orbbec-astra"/>
   <!-- no-add-on, lidar-back -->
   <xacro:arg name="add_on_module" default="lidar-back"/>
@@ -58,5 +58,6 @@
   <!-- HW configuration -->
   <xacro:property name="base_type" value="$(arg base_type)" />
-  <xacro:property name="head_type" value="$(arg head_type)" />
+  <xacro:property name="head_type" value="${'custom' if camera_model == 'azure-kinect' else 'original'}"/>
+  <!-- <xacro:property name="head_type" value="custom"/> -->
   <xacro:property name="laser_model" value="$(arg laser_model)" />
   <xacro:property name="arm_type" value="$(arg arm_type)" />
@@ -72,7 +73,4 @@
   <xacro:if value="${base_type not in ['pmb2', 'omni_base']}">
     <xacro:wrong_base_type/>
-  </xacro:if>
-  <xacro:if value="${head_type not in ['original', 'custom']}">
-    <xacro:wrong_head_type/>
   </xacro:if>
   <xacro:if value="${laser_model not in ['no-laser', 'sick-551', 'sick-561', 'sick-571', 'hokuyo']}">
@@ -93,7 +91,4 @@
   <xacro:if value="${camera_model not in ['no-camera', 'orbbec-astra', 'orbbec-astra-pro', 'asus-xtion', 'azure-kinect']}">
     <xacro:wrong_camera_model/>
-  </xacro:if>
-  <xacro:if value="${add_on_module not in ['no-add-on', 'lidar-back']}">
-    <xacro:wrong_add_on_module/>
   </xacro:if>
   <!-- HW configuration helpers-->

File: tiago_description/urdf/head/head_custom.urdf.xacro (robot description, xacro)
@@ -25,4 +25,5 @@
   <!-- INCLUDES -->
   <xacro:include filename="$(find pal_urdf_utils)/urdf/deg_to_rad.urdf.xacro" />
+  <xacro:include filename="$(find tiago_description)/urdf/sensors/orbbec_astra.urdf.xacro" />
   <xacro:include filename="$(find tiago_description)/urdf/sensors/azure_kinect.urdf.xacro" />
   <xacro:include filename="$(arg description_calibration_dir)/calibration_constants.urdf.xacro" />
@@ -32,5 +33,5 @@
     <link name="${name}_link">
       <inertial>
-        <origin xyz="-9.401 0.0 78.826" rpy="0.00000 0.00000 0.00000"/>
+        <origin xyz="-0.009401 0.0 0.078826" rpy="0.00000 0.00000 0.00000"/>
         <mass value="0.121"/>
         <inertia ixx="0.00035237400" ixy="-0.00000000100" ixz="0.00000793600" iyy="0.00038520500" iyz="-0.00000000500" izz="0.00028131647"/>
@@ -49,5 +50,5 @@
         </geometry>
         <material name="White" />
-      </collision>Head
+      </collision>
     </link>
     <joint name="${name}_joint" type="revolute">
@@ -105,8 +106,12 @@
     <xacro:head_1 name="${name}_1" parent="${parent}" />
     <xacro:head_2 name="${name}_2" parent="${name}_1_link"/>
+    <!-- Orbecc Astra Virtual -->
+    <xacro:orbbec_astra name="head_front_camera" parent="${name}_2_link" camera_model="orbbec-astra" extrinsic_calibration_dir="${extrinsic_calibration_dir}">
+      <origin xyz="${camera_position_x} ${camera_position_y} ${camera_position_z}" rpy="${camera_orientation_r} ${camera_orientation_p} ${camera_orientation_y}" />
+      <origin xyz="0 0 0" rpy="${-90 * deg_to_rad} ${0 * deg_to_rad} ${-90 * deg_to_rad}" />
+    </xacro:orbbec_astra>
     <!-- Azure Kinect -->
-    <!-- CHECK VALUES FROM CAMERA REAL NODE -->
+    <!-- Parent link frame to Kinect Screw Mount -->
     <xacro:azure_kinect name="azure_kinect" parent="${name}_2_link" xyz="0.0414 0.0725 0" rpy="${-90 * deg_to_rad} 0.0 0.0" >
-    <!-- Parent link frame to Kinect Screw Mount -->
     </xacro:azure_kinect>
   </xacro:macro>

Commit message: Added tray ee under custom ee

File: tiago_description/robots/tiago.urdf.xacro (robot description, xacro)
@@ -86,5 +86,5 @@
     <xacro:wrong_wrist_model/>
   </xacro:if>
-  <xacro:if value="${end_effector not in ['no-end-effector', 'pal-gripper', 'pal-hey5', 'custom', 'robotiq-2f-85', 'robotiq-2f-140']}">
+  <xacro:if value="${end_effector not in ['no-end-effector', 'pal-gripper', 'pal-hey5', 'custom', 'robotiq-2f-85', 'robotiq-2f-140', 'tray']}">
     <xacro:wrong_end_effector/>
   </xacro:if>

File: tiago_description/urdf/end_effector/end_effector.urdf.xacro (robot description, xacro)
@@ -33,4 +33,15 @@
         <origin xyz="0.01 0 0" rpy="${90*deg_to_rad} ${90*deg_to_rad} ${-90*deg_to_rad}"/>
       </xacro:pal_gripper>
+    </xacro:if>
+    <!-- PAL Gripper custom add-ons -->
+    <xacro:if value="${end_effector == 'custom'}">
+      <xacro:include filename="$(find pal_gripper_description)/urdf/gripper.urdf.xacro" />
+      <xacro:pal_gripper parent="${parent}" name="${name}">
+        <origin xyz="0.01 0 0" rpy="${90*deg_to_rad} ${90*deg_to_rad} ${-90*deg_to_rad}"/>
+      </xacro:pal_gripper>
+      <xacro:include filename="$(find tiago_description)/urdf/end_effector/tray_end_effector_add_on.urdf.xacro" />
+      <xacro:tray_end_effector_add_on name="tray_end_effector_add_on" parent="gripper_link" >
+        <origin xyz="0.0 -0.04 -0.125" rpy="${0*deg_to_rad} ${90*deg_to_rad} ${-90*deg_to_rad}"/>
+      </xacro:tray_end_effector_add_on>
     </xacro:if>
     <!-- Robotiq 2F-85 Gripper -->

File: tiago_description/urdf/sensors/orbbec_astra_virtual.urdf.xacro (robot description, xacro)
@@ -27,5 +27,5 @@
     <link name="${name}_link">
       <inertial>
-        <origin xyz="-0.00936000000 -0.00003000000 -0.00273000000" rpy="0 0 0"/>
+        <origin xyz="0.0 0.0 0.0" rpy="0 0 0"/>
         <mass value="0.001"/>
         <inertia ixx="0.00001" ixy="0" ixz="0" iyy="0.00001" iyz="0" izz="0.00001"/>

Commit message: Hardcoded new head to use it on TIAGo

File: tiago_description/robots/tiago.urdf.xacro (robot description, xacro)
@@ -58,6 +58,6 @@
   <!-- HW configuration -->
   <xacro:property name="base_type" value="$(arg base_type)" />
-  <xacro:property name="head_type" value="${'custom' if camera_model == 'azure-kinect' else 'original'}"/>
-  <!-- <xacro:property name="head_type" value="custom"/> -->
+  <!-- <xacro:property name="head_type" value="${'custom' if camera_model == 'azure-kinect' else 'original'}"/> -->
+  <xacro:property name="head_type" value="custom"/>
   <xacro:property name="laser_model" value="$(arg laser_model)" />
   <xacro:property name="arm_type" value="$(arg arm_type)" />
@@ -65,5 +65,6 @@
   <xacro:property name="wrist_model" value="$(arg wrist_model)" />
   <xacro:property name="end_effector" value="$(arg end_effector)" />
-  <xacro:property name="camera_model" value="$(arg camera_model)" />
+  <!-- <xacro:property name="camera_model" value="$(arg camera_model)" /> -->
+  <xacro:property name="camera_model" value="azure-kinect" />
   <xacro:property name="has_thermal_camera" default="$(arg has_thermal_camera)"/>
   <xacro:property name="has_screen" value="$(arg has_screen)" />
